File: electronics/flightcontroller/mcu.kicad_sch (KiCad schematic)
At the start: 31 parts, among them J10 USB, J8 Micro_SD_Card_Det_HYC80-TF08-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, J9 SWD, SW1 RESET, U3 STM32G491CCUx, U6 GT-24-Mini, Y1 24MHz

Commit message: electronics: Placed missing resistors and fixed remaining DRC errors.
Parts:
- added R24, R25: 47k, Resistor_SMD:R_0402_1005Metric, symbol Device:R
Connections:
- net +3V3: now also R24.1, R25.1
- net at J8.8 (DAT1), TP2.1: now also R24.2
- net at J8.1 (DAT2): now also R25.2
- no-connect marks 12 -> 11
Other:
- moved on the sheet: C27, C28, J8, TP2, Y1
