File: electronics/flightcontroller/sensors.kicad_sch (KiCad schematic)
At the start: 12 parts, among them U2 MPU-9250

Commit message: electronics: Changed the 4V regulator and added some ordering codes.
Parts:
- C10, C9: Mouser (none) -> 81-GRM155R61H104KE4D
- C21, C22: renamed from C?; Mouser (none) -> 81-GRM155R61H104KE4D
- C23, C24, C25, C26: renamed from C?; value 1uF/6.3V -> 10uF/6.3V; Digikey (none) -> 490-GRM155R60J106ME05DCT-ND
- gave numbers to parts that had none: 3
Changed lines of the file:
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@@
   (symbol (lib_id "power:+3.3V") (at 62.23 124.46 0) (unit 1)
     (in_bom yes) (on_board yes) (fields_autoplaced)
-    (property "Reference" "#PWR?" (id 0) (at 62.23 128.27 0)
+    (property "Reference" "#PWR02" (id 0) (at 62.23 128.27 0)
       (effects (font (size 1.27 1.27)) hide)
     )
@@
   (symbol (lib_id "power:+3.3V") (at 243.84 69.85 0) (unit 1)
     (in_bom yes) (on_board yes) (fields_autoplaced)
-    (property "Reference" "#PWR?" (id 0) (at 243.84 73.66 0)
+    (property "Reference" "#PWR04" (id 0) (at 243.84 73.66 0)
       (effects (font (size 1.27 1.27)) hide)
     )
@@
   (symbol (lib_id "power:+3.3V") (at 243.84 120.65 0) (unit 1)
     (in_bom yes) (on_board yes) (fields_autoplaced)
-    (property "Reference" "#PWR?" (id 0) (at 243.84 124.46 0)
+    (property "Reference" "#PWR06" (id 0) (at 243.84 124.46 0)
       (effects (font (size 1.27 1.27)) hide)
     )
@@
   (symbol (lib_id "power:GND") (at 77.47 142.24 0) (unit 1)
     (in_bom yes) (on_board yes) (fields_autoplaced)
-    (property "Reference" "#PWR?" (id 0) (at 77.47 148.59 0)
+    (property "Reference" "#PWR03" (id 0) (at 77.47 148.59 0)
       (effects (font (size 1.27 1.27)) hide)
     )
@@
   (symbol (lib_id "power:GND") (at 243.84 105.41 0) (unit 1)
     (in_bom yes) (on_board yes) (fields_autoplaced)
-    (property "Reference" "#PWR?" (id 0) (at 243.84 111.76 0)
+    (property "Reference" "#PWR05" (id 0) (at 243.84 111.76 0)
       (effects (font (size 1.27 1.27)) hide)
     )
@@
   (symbol (lib_id "power:GND") (at 243.84 156.21 0) (unit 1)
     (in_bom yes) (on_board yes) (fields_autoplaced)
-    (property "Reference" "#PWR?" (id 0) (at 243.84 162.56 0)
+    (property "Reference" "#PWR07" (id 0) (at 243.84 162.56 0)
       (effects (font (size 1.27 1.27)) hide)
     )
@@
   (symbol (lib_id "power:GND") (at 251.46 87.63 0) (unit 1)
     (in_bom yes) (on_board yes) (fields_autoplaced)
-    (property "Reference" "#PWR?" (id 0) (at 251.46 93.98 0)
+    (property "Reference" "#PWR08" (id 0) (at 251.46 93.98 0)
       (effects (font (size 1.27 1.27)) hide)
     )
@@
   (symbol (lib_id "power:GND") (at 251.46 138.43 0) (unit 1)
     (in_bom yes) (on_board yes) (fields_autoplaced)
-    (property "Reference" "#PWR?" (id 0) (at 251.46 144.78 0)
+    (property "Reference" "#PWR09" (id 0) (at 251.46 144.78 0)
       (effects (font (size 1.27 1.27)) hide)
     )
@@
   (symbol (lib_id "Device:R") (at 212.09 100.33 0) (unit 1)
     (in_bom yes) (on_board yes)
-    (property "Reference" "R?" (id 0) (at 208.28 99.0599 0)
+    (property "Reference" "R4" (id 0) (at 208.28 99.0599 0)
       (effects (font (size 1.27 1.27)) (justify left))
     )
@@
   (symbol (lib_id "Device:C") (at 77.47 133.35 0) (unit 1)
     (in_bom yes) (on_board yes) (fields_autoplaced)
-    (property "Reference" "C?" (id 0) (at 81.28 132.0799 0)
+    (property "Reference" "C21" (id 0) (at 81.28 132.0799 0)
       (effects (font (size 1.27 1.27)) (justify left))
     )
@@
       (effects (font (size 1.27 1.27)) hide)
     )
+    (property "Mouser" "81-GRM155R61H104KE4D" (id 4) (at 77.47 133.35 0)
+      (effects (font (size 1.27 1.27)) hide)
+    )
     (pin "1")
     (pin "2")
@@
       (effects (font (size 1.27 1.27)) hide)
     )
+    (property "Mouser" "81-GRM155R61H104KE4D" (id 4) (at 85.09 171.45 0)
+      (effects (font (size 1.27 1.27)) hide)
+    )
     (pin "1")
     (pin "2")
@@
   (symbol (lib_id "Device:C") (at 90.17 133.35 0) (unit 1)
     (in_bom yes) (on_board yes) (fields_autoplaced)
-    (property "Reference" "C?" (id 0) (at 93.98 132.0799 0)
+    (property "Reference" "C22" (id 0) (at 93.98 132.0799 0)
       (effects (font (size 1.27 1.27)) (justify left))
     )
@@
       (effects (font (size 1.27 1.27)) hide)
     )
+    (property "Mouser" "81-GRM155R61H104KE4D" (id 4) (at 90.17 133.35 0)
+      (effects (font (size 1.27 1.27)) hide)
+    )
     (pin "1")
     (pin "2")
@@
       (effects (font (size 1.27 1.27)) hide)
     )
+    (property "Mouser" "81-GRM155R61H104KE4D" (id 4) (at 97.79 171.45 0)
+      (effects (font (size 1.27 1.27)) hide)
+    )
     (pin "1")
     (pin "2")
@@
   (symbol (lib_id "Device:C") (at 251.46 78.74 0) (unit 1)
     (in_bom yes) (on_board yes) (fields_autoplaced)
-    (property "Reference" "C?" (id 0) (at 255.27 77.4699 0)
-      (effects (font (size 1.27 1.27)) (justify left))
-    )
-    (property "Value" "1uF/6.3V" (id 1) (at 255.27 80.0099 0)
+    (property "Reference" "C23" (id 0) (at 255.27 77.4699 0)
+      (effects (font (size 1.27 1.27)) (justify left))
+    )
+    (property "Value" "10uF/6.3V" (id 1) (at 255.27 80.0099 0)
       (effects (font (size 1.27 1.27)) (justify left))
     )
@@
       (effects (font (size 1.27 1.27)) hide)
     )
+    (property "Digikey" "490-GRM155R60J106ME05DCT-ND" (id 4) (at 251.46 78.74 0)
+      (effects (font (size 1.27 1.27)) hide)
+    )
     (pin "1")
     (pin "2")
@@
   (symbol (lib_id "Device:C") (at 251.46 129.54 0) (unit 1)
     (in_bom yes) (on_board yes) (fields_autoplaced)
-    (property "Reference" "C?" (id 0) (at 255.27 128.2699 0)
-      (effects (font (size 1.27 1.27)) (justify left))
-    )
-    (property "Value" "1uF/6.3V" (id 1) (at 255.27 130.8099 0)
+    (property "Reference" "C24" (id 0) (at 255.27 128.2699 0)
+      (effects (font (size 1.27 1.27)) (justify left))
+    )
+    (property "Value" "10uF/6.3V" (id 1) (at 255.27 130.8099 0)
       (effects (font (size 1.27 1.27)) (justify left))
     )
@@
       (effects (font (size 1.27 1.27)) hide)
     )
+    (property "Digikey" "490-GRM155R60J106ME05DCT-ND" (id 4) (at 251.46 129.54 0)
+      (effects (font (size 1.27 1.27)) hide)
+    )
     (pin "1")
     (pin "2")
@@
   (symbol (lib_id "Device:C") (at 267.97 78.74 0) (unit 1)
     (in_bom yes) (on_board yes) (fields_autoplaced)
-    (property "Reference" "C?" (id 0) (at 271.78 77.4699 0)
-      (effects (font (size 1.27 1.27)) (justify left))
-    )
-    (property "Value" "1uF/6.3V" (id 1) (at 271.78 80.0099 0)
+    (property "Reference" "C25" (id 0) (at 271.78 77.4699 0)
+      (effects (font (size 1.27 1.27)) (justify left))
+    )
+    (property "Value" "10uF/6.3V" (id 1) (at 271.78 80.0099 0)
       (effects (font (size 1.27 1.27)) (justify left))
     )
@@
       (effects (font (size 1.27 1.27)) hide)
     )
+    (property "Digikey" "490-GRM155R60J106ME05DCT-ND" (id 4) (at 267.97 78.74 0)
+      (effects (font (size 1.27 1.27)) hide)
+    )
     (pin "1")
     (pin "2")
@@
   (symbol (lib_id "Device:C") (at 267.97 129.54 0) (unit 1)
     (in_bom yes) (on_board yes) (fields_autoplaced)
-    (property "Reference" "C?" (id 0) (at 271.78 128.2699 0)
-      (effects (font (size 1.27 1.27)) (justify left))
-    )
-    (property "Value" "1uF/6.3V" (id 1) (at 271.78 130.8099 0)
+    (property "Reference" "C26" (id 0) (at 271.78 128.2699 0)
+      (effects (font (size 1.27 1.27)) (justify left))
+    )
+    (property "Value" "10uF/6.3V" (id 1) (at 271.78 130.8099 0)
       (effects (font (size 1.27 1.27)) (justify left))
     )
@@
     )
     (property "Datasheet" "~" (id 3) (at 267.97 129.54 0)
+      (effects (font (size 1.27 1.27)) hide)
+    )
+    (property "Digikey" "490-GRM155R60J106ME05DCT-ND" (id 4) (at 267.97 129.54 0)
       (effects (font (size 1.27 1.27)) hide)
     )
@@
   (symbol (lib_id "flightcontroller-symbols:Omron_2SMPB-02B") (at 238.76 88.9 0) (unit 1)
     (in_bom yes) (on_board yes)
-    (property "Reference" "U?" (id 0) (at 232.41 77.4699 0)
+    (property "Reference" "U7" (id 0) (at 232.41 77.4699 0)
       (effects (font (size 1.27 1.27)) (justify left))
     )
@@
   (symbol (lib_id "flightcontroller-symbols:Omron_2SMPB-02B") (at 238.76 139.7 0) (unit 1)
     (in_bom yes) (on_board yes)
-    (property "Reference" "U?" (id 0) (at 232.41 128.2699 0)
-      (effects (font (size 1.27 1.27)) (justify left))
-    )
+    (property "Reference" "U8" (id 0) (at 232.41 128.2699 0)
+      (effects (font (size 1.27 1.27)) (justify left))
+    )

Commit message: PCB: USB, micro SD, and many component changes.
Parts:
- C10, C21, C22, C9: Mouser 81-GRM155R61H104KE4D -> 81-GRM155R71H104KE4D
- C23, C24, C25, C26: footprint (none) -> Capacitor_SMD:C_0402_1005Metric; Digikey 490-GRM155R60J106ME05DCT-ND -> (none); Mouser (none) -> 81-GRM155R60J106M05D
- U7, U8: footprint (none) -> flightcontroller-footprints:Omron_2SMPB
Changed lines of the file:
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@@
       (effects (font (size 1.27 1.27)) hide)
     )
-    (property "Mouser" "81-GRM155R61H104KE4D" (id 4) (at 77.47 133.35 0)
+    (property "Mouser" "81-GRM155R71H104KE4D" (id 4) (at 77.47 133.35 0)
       (effects (font (size 1.27 1.27)) hide)
     )
@@
       (effects (font (size 1.27 1.27)) hide)
     )
-    (property "Mouser" "81-GRM155R61H104KE4D" (id 4) (at 85.09 171.45 0)
+    (property "Mouser" "81-GRM155R71H104KE4D" (id 4) (at 85.09 171.45 0)
       (effects (font (size 1.27 1.27)) hide)
     )
@@
       (effects (font (size 1.27 1.27)) hide)
     )
-    (property "Mouser" "81-GRM155R61H104KE4D" (id 4) (at 90.17 133.35 0)
+    (property "Mouser" "81-GRM155R71H104KE4D" (id 4) (at 90.17 133.35 0)
       (effects (font (size 1.27 1.27)) hide)
     )
@@
       (effects (font (size 1.27 1.27)) hide)
     )
-    (property "Mouser" "81-GRM155R61H104KE4D" (id 4) (at 97.79 171.45 0)
+    (property "Mouser" "81-GRM155R71H104KE4D" (id 4) (at 97.79 171.45 0)
       (effects (font (size 1.27 1.27)) hide)
     )
@@
       (effects (font (size 1.27 1.27)) (justify left))
     )
-    (property "Footprint" "" (id 2) (at 252.4252 82.55 0)
+    (property "Footprint" "Capacitor_SMD:C_0402_1005Metric" (id 2) (at 252.4252 82.55 0)
       (effects (font (size 1.27 1.27)) hide)
     )
@@
       (effects (font (size 1.27 1.27)) hide)
     )
-    (property "Digikey" "490-GRM155R60J106ME05DCT-ND" (id 4) (at 251.46 78.74 0)
+    (property "Digikey" "" (id 4) (at 251.46 78.74 0)
+      (effects (font (size 1.27 1.27)) hide)
+    )
+    (property "Mouser" "81-GRM155R60J106M05D" (id 5) (at 251.46 78.74 0)
       (effects (font (size 1.27 1.27)) hide)
     )
@@
       (effects (font (size 1.27 1.27)) (justify left))
     )
-    (property "Footprint" "" (id 2) (at 252.4252 133.35 0)
+    (property "Footprint" "Capacitor_SMD:C_0402_1005Metric" (id 2) (at 252.4252 133.35 0)
       (effects (font (size 1.27 1.27)) hide)
     )
@@
       (effects (font (size 1.27 1.27)) hide)
     )
-    (property "Digikey" "490-GRM155R60J106ME05DCT-ND" (id 4) (at 251.46 129.54 0)
+    (property "Digikey" "" (id 4) (at 251.46 129.54 0)
+      (effects (font (size 1.27 1.27)) hide)
+    )
+    (property "Mouser" "81-GRM155R60J106M05D" (id 5) (at 251.46 129.54 0)
       (effects (font (size 1.27 1.27)) hide)
     )
@@
       (effects (font (size 1.27 1.27)) (justify left))
     )
-    (property "Footprint" "" (id 2) (at 268.9352 82.55 0)
+    (property "Footprint" "Capacitor_SMD:C_0402_1005Metric" (id 2) (at 268.9352 82.55 0)
       (effects (font (size 1.27 1.27)) hide)
     )
@@
       (effects (font (size 1.27 1.27)) hide)
     )
-    (property "Digikey" "490-GRM155R60J106ME05DCT-ND" (id 4) (at 267.97 78.74 0)
+    (property "Digikey" "" (id 4) (at 267.97 78.74 0)
+      (effects (font (size 1.27 1.27)) hide)
+    )
+    (property "Mouser" "81-GRM155R60J106M05D" (id 5) (at 267.97 78.74 0)
       (effects (font (size 1.27 1.27)) hide)
     )
@@
       (effects (font (size 1.27 1.27)) (justify left))
     )
-    (property "Footprint" "" (id 2) (at 268.9352 133.35 0)
+    (property "Footprint" "Capacitor_SMD:C_0402_1005Metric" (id 2) (at 268.9352 133.35 0)
       (effects (font (size 1.27 1.27)) hide)
     )
@@
       (effects (font (size 1.27 1.27)) hide)
     )
-    (property "Digikey" "490-GRM155R60J106ME05DCT-ND" (id 4) (at 267.97 129.54 0)
-      (effects (font (size 1.27 1.27)) hide)
-    )
-    (pin "1")
-    (pin "2")
-  )
-  (symbol (lib_id "flightcontroller-symbols:Omron_2SMPB-02B") (at 238.76 88.9 0) (unit 1)
+    (property "Digikey" "" (id 4) (at 267.97 129.54 0)
+      (effects (font (size 1.27 1.27)) hide)
+    )
+    (property "Mouser" "81-GRM155R60J106M05D" (id 5) (at 267.97 129.54 0)
+      (effects (font (size 1.27 1.27)) hide)
+    )
+    (pin "1")
+    (pin "2")
+  )
+  (symbol (lib_name "Omron_2SMPB-02B_1") (lib_id "flightcontroller-symbols:Omron_2SMPB-02B") (at 238.76 88.9 0) (unit 1)
     (in_bom yes) (on_board yes)
     (property "Reference" "U7" (id 0) (at 232.41 77.4699 0)
@@
       (effects (font (size 1.27 1.27)) (justify left))
     )
-    (property "Footprint" "" (id 2) (at 238.76 88.9 0)
+    (property "Footprint" "flightcontroller-footprints:Omron_2SMPB" (id 2) (at 238.76 88.9 0)
       (effects (font (size 1.27 1.27)) hide)
     )
@@
     (pin "7")
     (pin "8")
-    (pin "9")
   )
   (symbol (lib_id "flightcontroller-symbols:Omron_2SMPB-02B") (at 238.76 139.7 0) (unit 1)
@@
       (effects (font (size 1.27 1.27)) (justify left))
     )
-    (property "Footprint" "" (id 2) (at 238.76 139.7 0)
+    (property "Footprint" "flightcontroller-footprints:Omron_2SMPB" (id 2) (at 238.76 139.7 0)
       (effects (font (size 1.27 1.27)) hide)
     )
@@
     (pin "7")
     (pin "8")
-    (pin "9")
   )
   (symbol (lib_id "Sensor_Motion:MPU-9250") (at 59.69 157.48 0) (unit 1)
