File: electronics/flightcontroller/sensors.kicad_sch (KiCad schematic)
At the start: 12 parts, among them U2 MPU-9250, U7 Omron_2SMPB-02B, U8 Omron_2SMPB-02B

Commit message: electronics: General PCB layout and size, let pressure sensors use I2C.
Parts:
- added R13: 10k, Resistor_SMD:R_0402_1005Metric, symbol Device:R
- R4: value 330 -> 10k
Connections:
- net PR1_~{CS} is gone; now on net +3V3: U7.2 (~{CS}/VDDIO), U8.2 (~{CS}/VDDIO)
- net +3V3: now also R13.1
- net GND: now also R4.2
- net at U8.5 (SDO/ADDR): now also R13.2; no longer R4.2
- net PR_RST: now reaches U7.1 (RST), U8.1 (RST)
- net PR_MISO: no longer names the net of R4.1, U7.5 (SDO/ADDR)
- net PR_MOSI renamed PR_SDA
- net PR_SCK renamed PR_SCL
Other:
- moved on the sheet: R4
Changed lines of the file:
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@@
   (junction (at 77.47 139.7) (diameter 0.9144) (color 0 0 0 0))
   (junction (at 80.01 177.8) (diameter 0.9144) (color 0 0 0 0))
-  (junction (at 212.09 93.98) (diameter 0.9144) (color 0 0 0 0))
-  (junction (at 214.63 91.44) (diameter 0.9144) (color 0 0 0 0))
-  (junction (at 217.17 88.9) (diameter 0.9144) (color 0 0 0 0))
+  (junction (at 207.01 91.44) (diameter 0.9144) (color 0 0 0 0))
+  (junction (at 209.55 88.9) (diameter 0.9144) (color 0 0 0 0))
+  (junction (at 212.09 81.28) (diameter 0.9144) (color 0 0 0 0))
+  (junction (at 241.3 72.39) (diameter 0.9144) (color 0 0 0 0))
+  (junction (at 241.3 123.19) (diameter 0.9144) (color 0 0 0 0))
   (junction (at 243.84 72.39) (diameter 0.9144) (color 0 0 0 0))
   (junction (at 243.84 123.19) (diameter 0.9144) (color 0 0 0 0))
@@
     (stroke (width 0) (type solid) (color 0 0 0 0))
   )
-  (wire (pts (xy 209.55 86.36) (xy 227.33 86.36))
-    (stroke (width 0) (type solid) (color 0 0 0 0))
-  )
-  (wire (pts (xy 209.55 88.9) (xy 217.17 88.9))
-    (stroke (width 0) (type solid) (color 0 0 0 0))
-  )
-  (wire (pts (xy 209.55 91.44) (xy 214.63 91.44))
-    (stroke (width 0) (type solid) (color 0 0 0 0))
-  )
-  (wire (pts (xy 209.55 93.98) (xy 212.09 93.98))
-    (stroke (width 0) (type solid) (color 0 0 0 0))
-  )
-  (wire (pts (xy 209.55 137.16) (xy 227.33 137.16))
-    (stroke (width 0) (type solid) (color 0 0 0 0))
-  )
-  (wire (pts (xy 212.09 93.98) (xy 212.09 96.52))
-    (stroke (width 0) (type solid) (color 0 0 0 0))
-  )
-  (wire (pts (xy 212.09 104.14) (xy 212.09 144.78))
-    (stroke (width 0) (type solid) (color 0 0 0 0))
-  )
-  (wire (pts (xy 212.09 144.78) (xy 227.33 144.78))
-    (stroke (width 0) (type solid) (color 0 0 0 0))
-  )
-  (wire (pts (xy 214.63 91.44) (xy 227.33 91.44))
-    (stroke (width 0) (type solid) (color 0 0 0 0))
-  )
-  (wire (pts (xy 214.63 142.24) (xy 214.63 91.44))
-    (stroke (width 0) (type solid) (color 0 0 0 0))
-  )
-  (wire (pts (xy 217.17 88.9) (xy 217.17 139.7))
-    (stroke (width 0) (type solid) (color 0 0 0 0))
-  )
-  (wire (pts (xy 217.17 139.7) (xy 227.33 139.7))
-    (stroke (width 0) (type solid) (color 0 0 0 0))
-  )
-  (wire (pts (xy 219.71 81.28) (xy 227.33 81.28))
-    (stroke (width 0) (type solid) (color 0 0 0 0))
-  )
-  (wire (pts (xy 219.71 132.08) (xy 219.71 81.28))
-    (stroke (width 0) (type solid) (color 0 0 0 0))
-  )
-  (wire (pts (xy 227.33 88.9) (xy 217.17 88.9))
-    (stroke (width 0) (type solid) (color 0 0 0 0))
-  )
-  (wire (pts (xy 227.33 93.98) (xy 212.09 93.98))
-    (stroke (width 0) (type solid) (color 0 0 0 0))
-  )
-  (wire (pts (xy 227.33 132.08) (xy 219.71 132.08))
-    (stroke (width 0) (type solid) (color 0 0 0 0))
-  )
-  (wire (pts (xy 227.33 142.24) (xy 214.63 142.24))
+  (wire (pts (xy 201.93 81.28) (xy 212.09 81.28))
+    (stroke (width 0) (type solid) (color 0 0 0 0))
+  )
+  (wire (pts (xy 201.93 88.9) (xy 209.55 88.9))
+    (stroke (width 0) (type solid) (color 0 0 0 0))
+  )
+  (wire (pts (xy 201.93 91.44) (xy 207.01 91.44))
+    (stroke (width 0) (type solid) (color 0 0 0 0))
+  )
+  (wire (pts (xy 207.01 91.44) (xy 227.33 91.44))
+    (stroke (width 0) (type solid) (color 0 0 0 0))
+  )
+  (wire (pts (xy 207.01 142.24) (xy 207.01 91.44))
+    (stroke (width 0) (type solid) (color 0 0 0 0))
+  )
+  (wire (pts (xy 209.55 88.9) (xy 209.55 139.7))
+    (stroke (width 0) (type solid) (color 0 0 0 0))
+  )
+  (wire (pts (xy 209.55 139.7) (xy 227.33 139.7))
+    (stroke (width 0) (type solid) (color 0 0 0 0))
+  )
+  (wire (pts (xy 212.09 81.28) (xy 227.33 81.28))
+    (stroke (width 0) (type solid) (color 0 0 0 0))
+  )
+  (wire (pts (xy 212.09 132.08) (xy 212.09 81.28))
+    (stroke (width 0) (type solid) (color 0 0 0 0))
+  )
+  (wire (pts (xy 219.71 93.98) (xy 219.71 96.52))
+    (stroke (width 0) (type solid) (color 0 0 0 0))
+  )
+  (wire (pts (xy 219.71 104.14) (xy 219.71 106.68))
+    (stroke (width 0) (type solid) (color 0 0 0 0))
+  )
+  (wire (pts (xy 222.25 119.38) (xy 222.25 121.92))
+    (stroke (width 0) (type solid) (color 0 0 0 0))
+  )
+  (wire (pts (xy 222.25 129.54) (xy 222.25 144.78))
+    (stroke (width 0) (type solid) (color 0 0 0 0))
+  )
+  (wire (pts (xy 222.25 144.78) (xy 227.33 144.78))
+    (stroke (width 0) (type solid) (color 0 0 0 0))
+  )
+  (wire (pts (xy 224.79 72.39) (xy 241.3 72.39))
+    (stroke (width 0) (type solid) (color 0 0 0 0))
+  )
+  (wire (pts (xy 224.79 86.36) (xy 224.79 72.39))
+    (stroke (width 0) (type solid) (color 0 0 0 0))
+  )
+  (wire (pts (xy 224.79 123.19) (xy 241.3 123.19))
+    (stroke (width 0) (type solid) (color 0 0 0 0))
+  )
+  (wire (pts (xy 224.79 137.16) (xy 224.79 123.19))
+    (stroke (width 0) (type solid) (color 0 0 0 0))
+  )
+  (wire (pts (xy 227.33 86.36) (xy 224.79 86.36))
+    (stroke (width 0) (type solid) (color 0 0 0 0))
+  )
+  (wire (pts (xy 227.33 88.9) (xy 209.55 88.9))
+    (stroke (width 0) (type solid) (color 0 0 0 0))
+  )
+  (wire (pts (xy 227.33 93.98) (xy 219.71 93.98))
+    (stroke (width 0) (type solid) (color 0 0 0 0))
+  )
+  (wire (pts (xy 227.33 132.08) (xy 212.09 132.08))
+    (stroke (width 0) (type solid) (color 0 0 0 0))
+  )
+  (wire (pts (xy 227.33 137.16) (xy 224.79 137.16))
+    (stroke (width 0) (type solid) (color 0 0 0 0))
+  )
+  (wire (pts (xy 227.33 142.24) (xy 207.01 142.24))
     (stroke (width 0) (type solid) (color 0 0 0 0))
   )
@@
     (effects (font (size 1.27 1.27)) (justify left))
   )
-  (hierarchical_label "PR1_~{CS}" (shape input) (at 209.55 86.36 180)
-    (effects (font (size 1.27 1.27)) (justify right))
-  )
-  (hierarchical_label "PR_SCK" (shape input) (at 209.55 88.9 180)
-    (effects (font (size 1.27 1.27)) (justify right))
-  )
-  (hierarchical_label "PR_MOSI" (shape input) (at 209.55 91.44 180)
-    (effects (font (size 1.27 1.27)) (justify right))
-  )
-  (hierarchical_label "PR_MISO" (shape output) (at 209.55 93.98 180)
-    (effects (font (size 1.27 1.27)) (justify right))
-  )
-  (hierarchical_label "PR1_~{CS}" (shape input) (at 209.55 137.16 180)
+  (hierarchical_label "PR_RST" (shape input) (at 201.93 81.28 180)
+    (effects (font (size 1.27 1.27)) (justify right))
+  )
+  (hierarchical_label "PR_SCL" (shape bidirectional) (at 201.93 88.9 180)
+    (effects (font (size 1.27 1.27)) (justify right))
+  )
+  (hierarchical_label "PR_SDA" (shape bidirectional) (at 201.93 91.44 180)
     (effects (font (size 1.27 1.27)) (justify right))
   )
@@
     (pin "1")
   )
+  (symbol (lib_id "power:+3.3V") (at 222.25 119.38 0) (unit 1)
+    (in_bom yes) (on_board yes) (fields_autoplaced)
+    (property "Reference" "#PWR013" (id 0) (at 222.25 123.19 0)
+      (effects (font (size 1.27 1.27)) hide)
+    )
+    (property "Value" "+3.3V" (id 1) (at 222.25 114.3 0))
+    (property "Footprint" "" (id 2) (at 222.25 119.38 0)
+      (effects (font (size 1.27 1.27)) hide)
+    )
+    (property "Datasheet" "" (id 3) (at 222.25 119.38 0)
+      (effects (font (size 1.27 1.27)) hide)
+    )
+    (pin "1")
+  )
   (symbol (lib_id "power:+3.3V") (at 243.84 69.85 0) (unit 1)
     (in_bom yes) (on_board yes) (fields_autoplaced)
@@
     (pin "1")
   )
+  (symbol (lib_id "power:GND") (at 219.71 106.68 0) (unit 1)
+    (in_bom yes) (on_board yes) (fields_autoplaced)
+    (property "Reference" "#PWR012" (id 0) (at 219.71 113.03 0)
+      (effects (font (size 1.27 1.27)) hide)
+    )
+    (property "Value" "GND" (id 1) (at 219.71 111.76 0))
+    (property "Footprint" "" (id 2) (at 219.71 106.68 0)
+      (effects (font (size 1.27 1.27)) hide)
+    )
+    (property "Datasheet" "" (id 3) (at 219.71 106.68 0)
+      (effects (font (size 1.27 1.27)) hide)
+    )
+    (pin "1")
+  )
   (symbol (lib_id "power:GND") (at 243.84 105.41 0) (unit 1)
     (in_bom yes) (on_board yes) (fields_autoplaced)
@@
     (pin "1")
   )
-  (symbol (lib_id "Device:R") (at 212.09 100.33 0) (unit 1)
+  (symbol (lib_id "Device:R") (at 219.71 100.33 0) (unit 1)
     (in_bom yes) (on_board yes)
-    (property "Reference" "R4" (id 0) (at 208.28 99.0599 0)
+    (property "Reference" "R4" (id 0) (at 215.9 99.0599 0)
       (effects (font (size 1.27 1.27)) (justify left))
     )
-    (property "Value" "330" (id 1) (at 207.01 101.5999 0)
+    (property "Value" "10k" (id 1) (at 214.63 101.5999 0)
       (effects (font (size 1.27 1.27)) (justify left))
     )
-    (property "Footprint" "Resistor_SMD:R_0402_1005Metric" (id 2) (at 210.312 100.33 90)
-      (effects (font (size 1.27 1.27)) hide)
-    )
-    (property "Datasheet" "~" (id 3) (at 212.09 100.33 0)
-      (effects (font (size 1.27 1.27)) hide)
-    )
+    (property "Footprint" "Resistor_SMD:R_0402_1005Metric" (id 2) (at 217.932 100.33 90)
+      (effects (font (size 1.27 1.27)) hide)
+    )
+    (property "Datasheet" "~" (id 3) (at 219.71 100.33 0)
+      (effects (font (size 1.27 1.27)) hide)
+    )
+    (pin "1")
+    (pin "2")
+  )
+  (symbol (lib_id "Device:R") (at 222.25 125.73 0) (unit 1)
+    (in_bom yes) (on_board yes)
+    (property "Reference" "R13" (id 0) (at 218.44 124.4599 0)
+      (effects (font (size 1.27 1.27)) (justify left))
+    )
+    (property "Value" "10k" (id 1) (at 217.17 126.9999 0)
+      (effects (font (size 1.27 1.27)) (justify left))
+    )
+    (property "Footprint" "Resistor_SMD:R_0402_1005Metric" (id 2) (at 220.472 125.73 90)
+      (effects (font (size 1.27 1.27)) hide)
+    )
+    (property "Datasheet" "~" (id 3) (at 222.25 125.73 0)
+      (effects (font (size 1.27 1.27)) hide)
+    )

Commit message: electronics: Microcontroller connections, general component placement.
Parts:
- added R16, R18: 4.7k, Resistor_SMD:R_0402_1005Metric, symbol Device:R
- added R17: 10k, Resistor_SMD:R_0402_1005Metric, symbol Device:R
Connections:
- net +3V3: now also R16.1, R18.1
- net GND: now also R17.2
- net PR_RST: now also R17.1
- net PR_SCL: now also R18.2
- net PR_SDA: now also R16.2
Other:
- note added: "Pressure sensors for altitude and airspeed"
Changed lines of the file:
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@@
   (junction (at 209.55 88.9) (diameter 0.9144) (color 0 0 0 0))
   (junction (at 212.09 81.28) (diameter 0.9144) (color 0 0 0 0))
+  (junction (at 212.09 132.08) (diameter 0.9144) (color 0 0 0 0))
+  (junction (at 217.17 88.9) (diameter 0.9144) (color 0 0 0 0))
   (junction (at 241.3 72.39) (diameter 0.9144) (color 0 0 0 0))
   (junction (at 241.3 123.19) (diameter 0.9144) (color 0 0 0 0))
@@
     (stroke (width 0) (type solid) (color 0 0 0 0))
   )
+  (wire (pts (xy 207.01 68.58) (xy 207.01 71.12))
+    (stroke (width 0) (type solid) (color 0 0 0 0))
+  )
+  (wire (pts (xy 207.01 78.74) (xy 207.01 91.44))
+    (stroke (width 0) (type solid) (color 0 0 0 0))
+  )
   (wire (pts (xy 207.01 91.44) (xy 227.33 91.44))
     (stroke (width 0) (type solid) (color 0 0 0 0))
@@
     (stroke (width 0) (type solid) (color 0 0 0 0))
   )
+  (wire (pts (xy 212.09 132.08) (xy 212.09 144.78))
+    (stroke (width 0) (type solid) (color 0 0 0 0))
+  )
+  (wire (pts (xy 212.09 152.4) (xy 212.09 154.94))
+    (stroke (width 0) (type solid) (color 0 0 0 0))
+  )
+  (wire (pts (xy 217.17 68.58) (xy 217.17 71.12))
+    (stroke (width 0) (type solid) (color 0 0 0 0))
+  )
+  (wire (pts (xy 217.17 78.74) (xy 217.17 88.9))
+    (stroke (width 0) (type solid) (color 0 0 0 0))
+  )
+  (wire (pts (xy 217.17 88.9) (xy 209.55 88.9))
+    (stroke (width 0) (type solid) (color 0 0 0 0))
+  )
   (wire (pts (xy 219.71 93.98) (xy 219.71 96.52))
     (stroke (width 0) (type solid) (color 0 0 0 0))
@@
     (stroke (width 0) (type solid) (color 0 0 0 0))
   )
-  (wire (pts (xy 227.33 88.9) (xy 209.55 88.9))
+  (wire (pts (xy 227.33 88.9) (xy 217.17 88.9))
     (stroke (width 0) (type solid) (color 0 0 0 0))
   )
@@
   )
   (polyline (pts (xy 109.22 190.5) (xy 109.22 115.57))
+    (stroke (width 0) (type dash) (color 0 0 0 0))
+  )
+  (polyline (pts (xy 191.77 57.15) (xy 191.77 163.83))
+    (stroke (width 0) (type dash) (color 0 0 0 0))
+  )
+  (polyline (pts (xy 191.77 57.15) (xy 283.21 57.15))
+    (stroke (width 0) (type dash) (color 0 0 0 0))
+  )
+  (polyline (pts (xy 283.21 57.15) (xy 283.21 163.83))
+    (stroke (width 0) (type dash) (color 0 0 0 0))
+  )
+  (polyline (pts (xy 283.21 163.83) (xy 191.77 163.83))
     (stroke (width 0) (type dash) (color 0 0 0 0))
   )
@@
     (effects (font (size 1.27 1.27)) (justify left bottom))
   )
+  (text "Pressure sensors for altitude and airspeed" (at 193.04 60.96 0)
+    (effects (font (size 1.27 1.27)) (justify left bottom))
+  )
   (hierarchical_label "IMU_MOSI" (shape input) (at 39.37 149.86 180)
     (effects (font (size 1.27 1.27)) (justify right))
@@
     (pin "1")
   )
+  (symbol (lib_id "power:+3.3V") (at 207.01 68.58 0) (unit 1)
+    (in_bom yes) (on_board yes) (fields_autoplaced)
+    (property "Reference" "#PWR020" (id 0) (at 207.01 72.39 0)
+      (effects (font (size 1.27 1.27)) hide)
+    )
+    (property "Value" "+3.3V" (id 1) (at 207.01 63.5 0))
+    (property "Footprint" "" (id 2) (at 207.01 68.58 0)
+      (effects (font (size 1.27 1.27)) hide)
+    )
+    (property "Datasheet" "" (id 3) (at 207.01 68.58 0)
+      (effects (font (size 1.27 1.27)) hide)
+    )
+    (pin "1")
+  )
+  (symbol (lib_id "power:+3.3V") (at 217.17 68.58 0) (unit 1)
+    (in_bom yes) (on_board yes) (fields_autoplaced)
+    (property "Reference" "#PWR022" (id 0) (at 217.17 72.39 0)
+      (effects (font (size 1.27 1.27)) hide)
+    )
+    (property "Value" "+3.3V" (id 1) (at 217.17 63.5 0))
+    (property "Footprint" "" (id 2) (at 217.17 68.58 0)
+      (effects (font (size 1.27 1.27)) hide)
+    )
+    (property "Datasheet" "" (id 3) (at 217.17 68.58 0)
+      (effects (font (size 1.27 1.27)) hide)
+    )
+    (pin "1")
+  )
   (symbol (lib_id "power:+3.3V") (at 222.25 119.38 0) (unit 1)
     (in_bom yes) (on_board yes) (fields_autoplaced)
@@
     (pin "1")
   )
+  (symbol (lib_id "power:GND") (at 212.09 154.94 0) (unit 1)
+    (in_bom yes) (on_board yes) (fields_autoplaced)
+    (property "Reference" "#PWR021" (id 0) (at 212.09 161.29 0)
+      (effects (font (size 1.27 1.27)) hide)
+    )
+    (property "Value" "GND" (id 1) (at 212.09 160.02 0))
+    (property "Footprint" "" (id 2) (at 212.09 154.94 0)
+      (effects (font (size 1.27 1.27)) hide)
+    )
+    (property "Datasheet" "" (id 3) (at 212.09 154.94 0)
+      (effects (font (size 1.27 1.27)) hide)
+    )
+    (pin "1")
+  )
   (symbol (lib_id "power:GND") (at 219.71 106.68 0) (unit 1)
     (in_bom yes) (on_board yes) (fields_autoplaced)
@@
     )
     (pin "1")
+  )
+  (symbol (lib_id "Device:R") (at 207.01 74.93 0) (unit 1)
+    (in_bom yes) (on_board yes)
+    (property "Reference" "R16" (id 0) (at 201.93 73.6599 0)
+      (effects (font (size 1.27 1.27)) (justify left))
+    )
+    (property "Value" "4.7k" (id 1) (at 200.66 76.1999 0)
+      (effects (font (size 1.27 1.27)) (justify left))
+    )
+    (property "Footprint" "Resistor_SMD:R_0402_1005Metric" (id 2) (at 205.232 74.93 90)
+      (effects (font (size 1.27 1.27)) hide)
+    )
+    (property "Datasheet" "~" (id 3) (at 207.01 74.93 0)
+      (effects (font (size 1.27 1.27)) hide)
+    )
+    (pin "1")
+    (pin "2")
+  )
+  (symbol (lib_id "Device:R") (at 212.09 148.59 0) (unit 1)
+    (in_bom yes) (on_board yes)
+    (property "Reference" "R17" (id 0) (at 208.28 147.3199 0)
+      (effects (font (size 1.27 1.27)) (justify left))
+    )
+    (property "Value" "10k" (id 1) (at 207.01 149.8599 0)
+      (effects (font (size 1.27 1.27)) (justify left))
+    )
+    (property "Footprint" "Resistor_SMD:R_0402_1005Metric" (id 2) (at 210.312 148.59 90)
+      (effects (font (size 1.27 1.27)) hide)
+    )
+    (property "Datasheet" "~" (id 3) (at 212.09 148.59 0)
+      (effects (font (size 1.27 1.27)) hide)
+    )
+    (pin "1")
+    (pin "2")
+  )
+  (symbol (lib_id "Device:R") (at 217.17 74.93 0) (unit 1)
+    (in_bom yes) (on_board yes)
+    (property "Reference" "R18" (id 0) (at 212.09 73.6599 0)
+      (effects (font (size 1.27 1.27)) (justify left))
+    )
+    (property "Value" "4.7k" (id 1) (at 210.82 76.1999 0)
+      (effects (font (size 1.27 1.27)) (justify left))
+    )
+    (property "Footprint" "Resistor_SMD:R_0402_1005Metric" (id 2) (at 215.392 74.93 90)
+      (effects (font (size 1.27 1.27)) hide)
+    )
+    (property "Datasheet" "~" (id 3) (at 217.17 74.93 0)
+      (effects (font (size 1.27 1.27)) hide)
+    )
+    (pin "1")
+    (pin "2")
   )
   (symbol (lib_id "Device:R") (at 219.71 100.33 0) (unit 1)
@@
   (symbol (lib_id "Device:R") (at 222.25 125.73 0) (unit 1)
     (in_bom yes) (on_board yes)
-    (property "Reference" "R13" (id 0) (at 218.44 124.4599 0)
-      (effects (font (size 1.27 1.27)) (justify left))
-    )
+    (property "Reference" "R13" (id 0) (at 217.17 124.4599 0)
+      (effects (font (size 1.27 1.27)) (justify left))
+    )

Commit message: electronics: Fix remaining schematics ERC errors.
Connections:
- net GND: now also C10.2
Changed lines of the file:
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@@
+    (stroke (width 0) (type solid) (color 0 0 0 0))
+  )
+  (wire (pts (xy 97.79 177.8) (xy 97.79 175.26))
     (stroke (width 0) (type solid) (color 0 0 0 0))
   )
@@
     (pin "1")
   )
-  (symbol (lib_id "power:+3.3V") (at 97.79 160.02 0) (unit 1)
-    (in_bom yes) (on_board yes) (fields_autoplaced)
-    (property "Reference" "#PWR0118" (id 0) (at 97.79 163.83 0)
-      (effects (font (size 1.27 1.27)) hide)
-    )
-    (property "Value" "+3.3V" (id 1) (at 97.79 154.94 0))
-    (property "Footprint" "" (id 2) (at 97.79 160.02 0)
-      (effects (font (size 1.27 1.27)) hide)
-    )
-    (property "Datasheet" "" (id 3) (at 97.79 160.02 0)
-      (effects (font (size 1.27 1.27)) hide)
-    )
-    (pin "1")
-  )
   (symbol (lib_id "power:+3.3V") (at 207.01 68.58 0) (unit 1)
     (in_bom yes) (on_board yes) (fields_autoplaced)
@@
     )
     (property "Datasheet" "" (id 3) (at 80.01 180.34 0)
+      (effects (font (size 1.27 1.27)) hide)
+    )
+    (pin "1")
+  )
+  (symbol (lib_id "power:GND") (at 97.79 177.8 0) (unit 1)
+    (in_bom yes) (on_board yes) (fields_autoplaced)
+    (property "Reference" "#PWR0118" (id 0) (at 97.79 184.15 0)
+      (effects (font (size 1.27 1.27)) hide)
+    )
+    (property "Value" "GND" (id 1) (at 97.79 182.88 0))
+    (property "Footprint" "" (id 2) (at 97.79 177.8 0)
+      (effects (font (size 1.27 1.27)) hide)
+    )
+    (property "Datasheet" "" (id 3) (at 97.79 177.8 0)
       (effects (font (size 1.27 1.27)) hide)
     )
@@
     (pin "2")
   )
-  (symbol (lib_name "Omron_2SMPB-02B_1") (lib_id "flightcontroller-symbols:Omron_2SMPB-02B") (at 238.76 88.9 0) (unit 1)
+  (symbol (lib_id "flightcontroller-symbols:Omron_2SMPB-02B") (at 238.76 88.9 0) (unit 1)
     (in_bom yes) (on_board yes)
     (property "Reference" "U7" (id 0) (at 232.41 77.4699 0)

Commit message: electronics: Add a resistor for ESC power and some test pads.
Connections:
- net +3V3: now also C9.1, U2.1 (RESV_VDDIO)
Changed lines of the file:
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@@
   (junction (at 77.47 139.7) (diameter 0.9144) (color 0 0 0 0))
   (junction (at 80.01 177.8) (diameter 0.9144) (color 0 0 0 0))
+  (junction (at 85.09 165.1) (diameter 0) (color 0 0 0 0))
   (junction (at 207.01 91.44) (diameter 0.9144) (color 0 0 0 0))
   (junction (at 209.55 88.9) (diameter 0.9144) (color 0 0 0 0))
@@
     (stroke (width 0) (type solid) (color 0 0 0 0))
   )
+  (wire (pts (xy 85.09 160.02) (xy 85.09 165.1))
+    (stroke (width 0) (type default) (color 0 0 0 0))
+  )
   (wire (pts (xy 85.09 165.1) (xy 77.47 165.1))
     (stroke (width 0) (type solid) (color 0 0 0 0))
@@
     )
     (property "Datasheet" "" (id 3) (at 62.23 124.46 0)
+      (effects (font (size 1.27 1.27)) hide)
+    )
+    (pin "1")
+  )
+  (symbol (lib_id "power:+3.3V") (at 85.09 160.02 0) (unit 1)
+    (in_bom yes) (on_board yes) (fields_autoplaced)
+    (property "Reference" "#PWR0158" (id 0) (at 85.09 163.83 0)
+      (effects (font (size 1.27 1.27)) hide)
+    )
+    (property "Value" "+3.3V" (id 1) (at 85.09 154.94 0))
+    (property "Footprint" "" (id 2) (at 85.09 160.02 0)
+      (effects (font (size 1.27 1.27)) hide)
+    )
+    (property "Datasheet" "" (id 3) (at 85.09 160.02 0)
       (effects (font (size 1.27 1.27)) hide)
     )
@@
   (symbol (lib_id "Device:R") (at 212.09 148.59 0) (unit 1)
     (in_bom yes) (on_board yes)
-    (property "Reference" "R17" (id 0) (at 208.28 147.3199 0)
+    (property "Reference" "R17" (id 0) (at 207.01 147.3199 0)
       (effects (font (size 1.27 1.27)) (justify left))
     )
